File: rover_led_udp_controller_hw/MCU&LEDS.kicad_sch (KiCad schematic)
At the start: 71 parts, among them IC2 TXS0108E, J10 DO_OUT, J11 CO_OUT, J12 DO_IN, J13 CI_IN, J14 DO_OUT_2, J15 DI_IN_2, J16 CO_OUT_2, J17 CI_IN_2, J2 +24V_PAD, J3 IN_+5, J4 OUT_+5, J5 GND_IN, J6 GND_OUT, J7 GND_PAD, J8 GND_IN, J9 GND_OUT, U2 LMR51450SDRRR, U3 SY8089AAAC(SOT23-5), U4 ESP32-S3-WROOM-1-N8R8

Commit message: Polarity protection and TSV protection
Parts:
- added C5, C6: 4.7uF/50V/X7R/1210, Capacitor_SMD:C_1210_3225Metric, symbol ESP32-S3-DevKit-LiPo_Rev_B:C
- added D2: 15V/SOD-123, Diode_SMD:D_SOD-123, symbol Device:D_Zener
- added D3: SMBJ33A, Diode_SMD:D_SMB, symbol Device:D_TVS
- added F2: 2A/1206, Fuse:Fuse_1206_3216Metric, symbol Device:Fuse
- added Q2: P-MOS 60V/SOT-23, Package_TO_SOT_SMD:SOT-23, symbol Transistor_FET:Q_PMOS_GSD
- added R6: 100k/R0603, Resistor_SMD:R_0603_1608Metric_Pad0.98x0.95mm_HandSolder, symbol ESP32-S3-DevKit-LiPo_Rev_B:R
- R3: renamed from R2; value 100k/R0603 -> 100k/1%/R0603
- R8: renamed from R6; value 19.1k/R0603 -> 19.1k/1%/R0603
- R9: renamed from R8; value 220k/R0603 -> 220k/1%/R0603
- renumbered C6 to C10, C7 to C11, C8 to C12, C9 to C13, C10 to C14, C11 to C15, C12 to C16, C13 to C17, C16 to C19, C17 to C20, C19 to C21, C20 to C22, C21 to C23, C22 to C24, C14 to C3, C15 to C4, C3 to C7, C4 to C8, C5 to C9, D8 to D10, D9 to D11, D10 to D12, D11 to D13, D12 to D14, D2 to D4, D3 to D5, D4 to D6, D5 to D7, D6 to D8, D7 to D9, R7 to R11, R9 to R12, R15 to R13, R12 to R14, R13 to R15, R14 to R16, R5 to R2, R3 to R4, R4 to R5, R11 to R7, U4 to U3, U3 to U4
Connections:
- net +24V: now also C5.1, C6.1, D2.1 (K), D3.1 (A1), Q2.2 (S); no longer J2.1 (Pin_1)
- net GND: now also C5.2, C6.2, D3.2 (A2), R6.1
- new net: F2.1, J2.1 (Pin_1)
- new net: F2.2, Q2.3 (D)
- new net: D2.2 (A), Q2.1 (G), R6.2
Other:
- note added: "SK9822"
- note removed: "APA102"
- moved on the sheet: BUT2, C10, C11, C12, C13, C14, C15, C16, C17, C18, C19, C2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
