File: rover_led_udp_controller_hw/MCU&LEDS.kicad_sch (KiCad schematic)
At the start: 78 parts, among them IC2 TXS0108E, J10 DO_OUT, J11 CO_OUT, J12 DO_IN, J13 CI_IN, J14 DO_OUT_2, J15 DI_IN_2, J16 CO_OUT_2, J17 CI_IN_2, J2 +24V_PAD, J3 IN_+5, J4 OUT_+5, J5 GND_IN, J6 GND_OUT, J7 GND_PAD, J8 GND_IN, J9 GND_OUT, Q2 P-MOS 60V/SOT-23, U2 LMR51450SDRRR, U3 ESP32-S3-WROOM-1-N8R8, U4 SY8089AAAC(SOT23-5)

Commit message: Fix F-01, F-02
Parts:
- removed C23: 22uF/10V/X5R/0603, Capacitor_SMD:C_0603_1608Metric, symbol ESP32-S3-DevKit-LiPo_Rev_B:C
- removed C5, C6: 4.7uF/50V/X7R/1210, Capacitor_SMD:C_1210_3225Metric, symbol ESP32-S3-DevKit-LiPo_Rev_B:C
- removed IC2: TXS0108E, MechatronicsAcademy:PW_R-PDSO-G20, symbol MechatronicsAcademy:TXS0108E
- removed R14: 100k/R0603, Resistor_SMD:R_0603_1608Metric_Pad0.98x0.95mm_HandSolder, symbol ESP32-S3-DevKit-LiPo_Rev_B:R
- added C21: 22uF/10V/X5R/0603, Capacitor_SMD:C_1210_3225Metric, symbol ESP32-S3-DevKit-LiPo_Rev_B:C
- added U5: 74AHCT125, Package_SO:SOIC-14_3.9x8.7mm_P1.27mm, symbol 74xx:74AHCT125
- C7: value 100uF/50V -> 4.7uF/50V/X7R/1206; footprint Capacitor_SMD:CP_Elec_8x10.5 -> Capacitor_SMD:C_1206_3216Metric_Pad1.33x1.80mm_HandSolder; Fieldname2 Value2 -> (none); Fieldname3 Value3 -> (none); JLCPCB C6100609 -> TODO
- C8, C9: value 4.7uF/50V -> 4.7uF/50V/X7R/1206; footprint Capacitor_SMD:CP_Elec_4x5.7 -> Capacitor_SMD:C_1206_3216Metric_Pad1.33x1.80mm_HandSolder; Fieldname2 Value2 -> (none); Fieldname3 Value3 -> (none); JLCPCB C2163350 -> TODO
- renumbered C24 to C22, C21 to C23, C22 to C24, R9 to R10, R10 to R11, R15 to R14, R16 to R15, R11 to R9
Connections:
- net +3.3V: now also C21.1
- net +5V: now also U5.14 (VCC)
- net GND: now also C21.2, U5.1, U5.10, U5.12, U5.13, U5.4, U5.7 (GND), U5.9
- net GPIO11\FSPID(SPI3_MOSI): now also U5.5
- net GPIO12\FSPICLK(SPI3_CLK): now also U5.2
- net LED_SPI_CLK: now also U5.3
- net LED_SPI_MOSI: now also U5.6
- no-connect marks 44 -> 34
Other:
- moved on the sheet: C10, C11, C12, C13, C14, C15, C16, C17, C19, C2, C20, C22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

Commit message: PCB redesign
Parts:
- removed C8, C9: 4.7uF/50V/X7R/1206, Capacitor_SMD:C_1206_3216Metric_Pad1.33x1.80mm_HandSolder, symbol ESP32-S3-DevKit-LiPo_Rev_B:C
- added C6: 4.7uF/50V, Capacitor_SMD:CP_Elec_4x5.7, symbol ESP32-S3-DevKit-LiPo_Rev_B:C
- C19: renamed from C21; footprint Capacitor_SMD:C_1210_3225Metric -> Capacitor_Tantalum_SMD:CP_EIA-2012-12_Kemet-R_HandSolder
- C22: renamed from C24; footprint Capacitor_SMD:C_0603_1608Metric -> Capacitor_Tantalum_SMD:CP_EIA-2012-12_Kemet-R_HandSolder
- C7: value 4.7uF/50V/X7R/1206 -> 4.7uF/50V; footprint Capacitor_SMD:C_1206_3216Metric_Pad1.33x1.80mm_HandSolder -> Capacitor_SMD:CP_Elec_4x5.7
- renumbered C12 to C10, C13 to C11, C14 to C12, C15 to C13, C16 to C14, C17 to C15, C18 to C16, C19 to C17, C20 to C18, C22 to C20, C23 to C21, C10 to C8, C11 to C9
Connections:
- net +24V: now also C6.1
- net GND: now also C6.2
Other:
- moved on the sheet: C21, C22, U5E

Commit message: PCB redesign
Parts:
- added C5, C6: 4.7uF/50V/X7R/1210, Capacitor_SMD:C_1210_3225Metric, symbol ESP32-S3-DevKit-LiPo_Rev_B:C
- C13: renamed from C12; symbol ESP32-S3-DevKit-LiPo_Rev_B:C -> Device:C_Polarized_Small
- C14: renamed from C13; symbol ESP32-S3-DevKit-LiPo_Rev_B:C -> Device:C_Polarized_Small
- C19: renamed from C18; symbol ESP32-S3-DevKit-LiPo_Rev_B:C -> Device:C_Polarized_Small
- C20: renamed from C19; footprint Capacitor_Tantalum_SMD:CP_EIA-2012-12_Kemet-R_HandSolder -> Capacitor_SMD:C_0603_1608Metric
- C22: footprint Capacitor_Tantalum_SMD:CP_EIA-2012-12_Kemet-R_HandSolder -> Capacitor_SMD:C_0603_1608Metric
- C7: renamed from C6; value 4.7uF/50V -> 100uF/50V; footprint Capacitor_SMD:CP_Elec_4x5.7 -> Capacitor_SMD:CP_Elec_8x10.5; symbol ESP32-S3-DevKit-LiPo_Rev_B:C -> Device:C_Polarized_Small
- C8: renamed from C7; value 4.7uF/50V -> 4.7uF/50V/X7R/1210; footprint Capacitor_SMD:CP_Elec_4x5.7 -> Capacitor_SMD:C_1210_3225Metric
- L2: value 4.7uH -> 4.7uH/MWSA1003S
- renumbered C9 to C10, C10 to C11, C11 to C12, C14 to C15, C15 to C16, C16 to C17, C17 to C18, C20 to C21, C21 to C23, C8 to C9
Connections:
- net +24V: now also C5.2, C6.2
- net GND: now also C5.1, C6.1
- net GPIO0\BUT1 renamed GPIO0_BUT1
- net GPIO11\FSPID(SPI3_MOSI) renamed GPIO11_FSPID_SPI3_MOSI
- net GPIO12\FSPICLK(SPI3_CLK) renamed GPIO12_FSPICLK_SPI3_CLK
- net GPIO19\USB_D- renamed GPIO19_USB_DM
- net GPIO20\USB_D+ renamed GPIO20_USB_DP
- net GPIO5\PWR_SENS renamed GPIO5_PWR_SENS
Other:
- moved on the sheet: C18, C22, C23, D3, U5E

Commit message: PCB redesign
Parts:
- added C24: 100nF/50V/0603, Capacitor_SMD:C_0603_1608Metric, symbol ESP32-S3-DevKit-LiPo_Rev_B:C
- added R13: 10k/R0603, Resistor_SMD:R_0603_1608Metric_Pad0.98x0.95mm_HandSolder, symbol ESP32-S3-DevKit-LiPo_Rev_B:R
- renumbered R13 to R14, R14 to R15, R15 to R16
Connections:
- net +3.3V: now also R13.1
- net GND: now also C24.2
- net GPIO0_BUT1: now also C24.1, R13.2
Other:
- moved on the sheet: BUT2, R14, RST2

Commit message: PCB redesign
Other:
- moved on the sheet: R3, R8
Changed lines of the file:
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@@
 	)
 	(junction
+		(at 213.36 69.85)
+		(diameter 0)
+		(color 0 0 0 0)
+	)
+	(junction
 		(at 259.08 93.98)
 		(diameter 0)
@@
 	)
 	(junction
+		(at 213.36 93.98)
+		(diameter 0)
+		(color 0 0 0 0)
+	)
+	(junction
 		(at 106.68 64.77)
 		(diameter 0)
@@
 	)
 	(junction
-		(at 214.63 93.98)
-		(diameter 0)
-		(color 0 0 0 0)
-	)
-	(junction
 		(at 302.26 73.66)
 		(diameter 0)
@@
 	)
 	(junction
-		(at 214.63 69.85)
-		(diameter 0)
-		(color 0 0 0 0)
-	)
-	(junction
 		(at 71.12 64.77)
 		(diameter 0)
@@
 	(wire
 		(pts
-			(xy 214.63 69.85) (xy 222.25 69.85)
-		)
-		(stroke
-			(width 0)
-			(type default)
-		)
-	)
-	(wire
-		(pts
 			(xy 143.51 204.47) (xy 151.13 204.47)
 		)
@@
 	(wire
 		(pts
-			(xy 214.63 80.01) (xy 214.63 93.98)
+			(xy 213.36 80.01) (xy 213.36 93.98)
 		)
 		(stroke
@@
 	(wire
 		(pts
-			(xy 205.74 69.85) (xy 214.63 69.85)
+			(xy 205.74 69.85) (xy 213.36 69.85)
 		)
 		(stroke
@@
 	(wire
 		(pts
-			(xy 214.63 93.98) (xy 222.25 93.98)
-		)
-		(stroke
-			(width 0)
-			(type default)
-		)
-	)
-	(wire
-		(pts
 			(xy 140.97 124.46) (xy 140.97 129.54)
 		)
@@
 	(wire
 		(pts
-			(xy 214.63 109.22) (xy 214.63 115.57)
+			(xy 213.36 107.95) (xy 213.36 114.3)
 		)
 		(stroke
@@
 	(wire
 		(pts
-			(xy 214.63 93.98) (xy 214.63 101.6)
+			(xy 213.36 93.98) (xy 213.36 100.33)
 		)
 		(stroke
@@
 	(wire
 		(pts
+			(xy 213.36 69.85) (xy 222.25 69.85)
+		)
+		(stroke
+			(width 0)
+			(type default)
+		)
+	)
+	(wire
+		(pts
 			(xy 449.58 242.57) (xy 403.86 242.57)
 		)
@@
 	(wire
 		(pts
-			(xy 214.63 69.85) (xy 214.63 72.39)
+			(xy 213.36 69.85) (xy 213.36 72.39)
 		)
 		(stroke
@@
 	(wire
 		(pts
-			(xy 182.88 93.98) (xy 214.63 93.98)
+			(xy 182.88 93.98) (xy 213.36 93.98)
 		)
 		(stroke
@@
 	(wire
 		(pts
+			(xy 213.36 93.98) (xy 222.25 93.98)
+		)
+		(stroke
+			(width 0)
+			(type default)
+		)
+	)
+	(wire
+		(pts
 			(xy 62.23 326.39) (xy 66.04 326.39)
 		)
@@
 		)
 		(property "JLCPCB" "C77055"
-			(at 315.214 79.756 90)
+			(at 352.552 220.726 90)
 			(show_name no)
 			(do_not_autoplace no)
@@
 		(dnp no)
 		(property "Reference" "R4"
-			(at 224.79 76.454 90)
+			(at 220.218 71.882 90)
 			(show_name no)
 			(do_not_autoplace no)
@@
 		)
 		(property "Value" "1k/R0603"
-			(at 219.71 76.708 0)
+			(at 225.044 74.93 0)
 			(show_name no)
 			(do_not_autoplace no)
@@
 		)
 		(property "JLCPCB" "C110776"
-			(at 224.79 71.12 0)
+			(at 219.964 77.724 0)
 			(show_name no)
 			(do_not_autoplace no)
@@
 		)
 		(property "Value" "4.7uH/MWSA1003S"
-			(at 189.992 71.628 0)
+			(at 188.722 71.628 0)
 			(show_name no)
 			(do_not_autoplace no)
@@
 	(symbol
 		(lib_id "ESP32-S3-DevKit-LiPo_Rev_B:R")
-		(at 214.63 76.2 270)
+		(at 213.36 76.2 270)
 		(mirror x)
 		(unit 1)
@@
 		(dnp no)
 		(property "Reference" "R3"
-			(at 217.17 76.454 90)
+			(at 211.836 72.136 90)
 			(show_name no)
 			(do_not_autoplace no)
@@
 		)
 		(property "Value" "100k/1%/R0603"
-			(at 212.09 80.01 0)
+			(at 216.154 78.74 0)
 			(show_name no)
 			(do_not_autoplace no)
@@
 		)
 		(property "Footprint" "Resistor_SMD:R_0603_1608Metric_Pad0.98x0.95mm_HandSolder"
-			(at 214.63 77.978 90)
+			(at 213.36 77.978 90)
 			(hide yes)
 			(show_name no)
@@
 		)
 		(property "Datasheet" ""
-			(at 214.63 76.2 0)
+			(at 213.36 76.2 0)
 			(show_name no)
 			(do_not_autoplace no)
@@
 		)
 		(property "Description" ""
-			(at 214.63 76.2 0)
+			(at 213.36 76.2 0)
 			(show_name no)
 			(do_not_autoplace no)
@@
 		)
 		(property "JLCPCB" "C100048"
-			(at 215.646 83.566 0)
+			(at 212.09 85.09 0)
 			(show_name no)
 			(do_not_autoplace no)
@@
 		(dnp no)
 		(property "Reference" "R7"
-			(at 313.69 98.298 0)
+			(at 310.642 98.806 0)
 			(show_name no)
 			(do_not_autoplace no)
@@
 		)
 		(property "JLCPCB" "C95204"
-			(at 319.532 98.806 0)
+			(at 317.246 99.06 0)
 			(show_name no)
 			(do_not_autoplace no)
@@
 	(symbol
 		(lib_id "ESP32-S3-DevKit-LiPo_Rev_B:R")
-		(at 214.63 105.41 270)
+		(at 213.36 104.14 270)
 		(mirror x)
 		(unit 1)
@@
 		(dnp no)
 		(property "Reference" "R8"
-			(at 216.916 101.854 90)
+			(at 215.646 100.584 90)
 			(show_name no)
 			(do_not_autoplace no)
@@
 		)
 		(property "Value" "19.1k/1%/R0603"
-			(at 212.09 105.664 0)
+			(at 210.82 104.394 0)
 			(show_name no)
 			(do_not_autoplace no)
@@
 		)
 		(property "Footprint" "Resistor_SMD:R_0603_1608Metric_Pad0.98x0.95mm_HandSolder"
-			(at 214.63 107.188 90)
+			(at 213.36 105.918 90)
 			(hide yes)
 			(show_name no)
@@
 		)
 		(property "Datasheet" ""
-			(at 214.63 105.41 0)
+			(at 213.36 104.14 0)
 			(show_name no)
 			(do_not_autoplace no)
@@
 		)
 		(property "Description" ""
-			(at 214.63 105.41 0)
+			(at 213.36 104.14 0)
 			(show_name no)
 			(do_not_autoplace no)
@@
 		)
 		(property "JLCPCB" "C173754"
-			(at 217.17 107.696 0)
+			(at 215.9 106.426 0)
 			(show_name no)
 			(do_not_autoplace no)
@@
 	(symbol
 		(lib_id "ESP32-S3-DevKit-LiPo_Rev_B:GND")
-		(at 214.63 115.57 0)
+		(at 213.36 114.3 0)
 		(unit 1)
 		(body_style 1)
@@
 		(dnp no)
 		(property "Reference" "#PWR020"
-			(at 214.63 121.92 0)
+			(at 213.36 120.65 0)
 			(hide yes)
 			(show_name no)
@@
 		)
 		(property "Value" "GND"
-			(at 214.63 119.38 0)
+			(at 213.36 118.11 0)
 			(show_name no)
 			(do_not_autoplace no)
@@
 		)
 		(property "Footprint" ""
-			(at 214.63 115.57 0)
+			(at 213.36 114.3 0)
 			(show_name no)
 			(do_not_autoplace no)
@@
 		)
 		(property "Datasheet" ""
-			(at 214.63 115.57 0)
+			(at 213.36 114.3 0)
 			(show_name no)
 			(do_not_autoplace no)
@@
 		)
 		(property "Description" ""
-			(at 214.63 115.57 0)
+			(at 213.36 114.3 0)
 			(show_name no)
 			(do_not_autoplace no)

Commit message: Update
Parts:
- removed C5, C6: 4.7uF/50V/X7R/1210, Capacitor_SMD:C_1210_3225Metric, symbol ESP32-S3-DevKit-LiPo_Rev_B:C
- added C16: 100nF/10V/X5R/0603, Capacitor_SMD:C_0603_1608Metric, symbol ESP32-S3-DevKit-LiPo_Rev_B:C
- added C21: 100nF/50V/0603, Capacitor_SMD:C_0603_1608Metric, symbol ESP32-S3-DevKit-LiPo_Rev_B:C
- added R13, R15: 100/R0603, Resistor_SMD:R_0603_1608Metric_Pad0.98x0.95mm_HandSolder, symbol ESP32-S3-DevKit-LiPo_Rev_B:R
- added U6: USBLC6-2SC6, Package_TO_SOT_SMD:SOT-23-6, symbol Power_Protection:USBLC6-2SC6
- F2: value 2A/1206 -> 3A/50A/30V/1812; footprint Fuse:Fuse_1206_3216Metric -> Fuse:Fuse_1812_4532Metric_Pad1.30x3.40mm_HandSolder
- renumbered C12 to C10, C13 to C11, C14 to C12, C15 to C13, C16 to C14, C17 to C15, C18 to C17, C19 to C18, C20 to C19, C21 to C20, C7 to C5, C8 to C6, C9 to C7, C10 to C8, C11 to C9, J7 to J5, J5 to J6, J6 to J7, R13 to R14, R14 to R16, R15 to R17, R16 to R18
Connections:
- net +5V: now also C16.1, U6.5 (VBUS)
- net GND: now also C16.2, C21.2, U6.2 (GND)
- net GPIO11_FSPID_SPI3_MOSI: now also R15.1; no longer U5.5
- net GPIO12_FSPICLK_SPI3_CLK: now also R13.1; no longer U5.2
- net GPIO19_USB_DM: now also U6.6 (I/O1); no longer USB-C2.A7 (DN1), USB-C2.B7 (DN2)
- net GPIO20_USB_DP: now also U6.4 (I/O2); no longer USB-C2.A6 (DP1), USB-C2.B6 (DP2)
- net GPIO5_PWR_SENS: now also C21.1
- net at F2.2, Q2.3 (D): now also D3.1 (A1)
- net +24V: no longer names the net of C5.1, C6.1, C7.2, C8.2, D2.1 (K), Q2.2 (S), U2.10 (VIN), U2.11 (VIN), U2.12 (VIN), U2.9 (EN)
- net +24V: no longer D3.1 (A1)
- new net: R15.2, U5.5
- new net: R13.2, U5.2
- new net: U6.3 (I/O2), USB-C2.A6 (DP1), USB-C2.B6 (DP2)
- new net: U6.1 (I/O1), USB-C2.A7 (DN1), USB-C2.B7 (DN2)
Other:
- note added: "Do not use high voltage rated cap for low voltage bus"
- note added: "Review: 1. TVS on input, capacitor paralele with TVS https://www.pololu.com/product/5380 2. Revie input capacitors 3. Use low ESR elec_cap 4. Do not use how voltage rated cap for low voltage bus"
- moved on the sheet: C22, C23, C24, D2, D3, D4, F2, J2, J5, L2, Q2, R6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
