File: rover_led_udp_controller_hw/rover_led_udp_controller_hw.kicad_pcb (KiCad board)
At the start: 2 copper layers, 100 x 25 mm, 75 parts, among them IC2 TXS0108E, J10 DO_OUT, J11 CO_OUT, J12 DO_IN, J13 CI_IN, J14 DO_OUT_2, J15 DI_IN_2, J16 CO_OUT_2, J17 CI_IN_2, J2 +24V_PAD, J3 IN_+5, J4 OUT_+5, J5 GND_IN, J6 GND_OUT, J7 GND_PAD, J8 GND_IN, J9 GND_OUT, U2 LMR51450SDRRR, U3 SY8089AAAC(SOT23-5), U4 ESP32-S3-WROOM-1-N8R8

Commit message: PCB redesign
Parts:
- removed the C21 at (78.2, 88.8)
- removed the C3 at (141.5, 81.5)
- removed the C4 at (155.0, 82.5)
- removed C5: 4.7uF/50V, Capacitor_SMD:CP_Elec_4x5.7
- removed IC2: TXS0108E, MechatronicsAcademy:PW_R-PDSO-G20
- removed the R12 at (74.5, 87.2)
- added C19: 22uF/10V/X5R/0603, Capacitor_Tantalum_SMD:CP_EIA-2012-12_Kemet-R_HandSolder, B.Cu at (119.8, 78.0)
- added C6: 4.7uF/50V, Capacitor_SMD:CP_Elec_4x5.7, B.Cu at (138.7, 84.2)
- added C7: 4.7uF/50V, Capacitor_SMD:CP_Elec_4x5.7, B.Cu at (138.7, 77.2)
- added D2: 15V/SOD-123, Diode_SMD:D_SOD-123, B.Cu at (147.0, 80.0)
- added D3: SMBJ33A, Diode_SMD:D_SMB, B.Cu at (143.5, 77.5)
- added F2: 2A/1206, Fuse:Fuse_1206_3216Metric, B.Cu at (155.0, 79.2)
- added Q2: P-MOS 60V/SOT-23, Package_TO_SOT_SMD:SOT-23, B.Cu at (150.4, 79.2)
- added R6: 100k/R0603, Resistor_SMD:R_0603_1608Metric_Pad0.98x0.95mm_HandSolder, B.Cu at (149.4, 82.6)
- added U5: 74AHCT125, Package_SO:SOIC-14_3.9x8.7mm_P1.27mm, B.Cu at (77.0, 82.3)
- C22: renamed from C20; footprint Capacitor_SMD:C_0603_1608Metric -> Capacitor_Tantalum_SMD:CP_EIA-2012-12_Kemet-R_HandSolder
- R10: renamed from R8; value 220k/R0603 -> 220k/1%/R0603
- R3: renamed from R2; value 100k/R0603 -> 100k/1%/R0603
- R8: renamed from R6; value 19.1k/R0603 -> 19.1k/1%/R0603
- moved C20 21.0 mm to (98.2, 94.0)
- moved C11 7.78 mm to (134.7, 89.7)
- moved C10 7.53 mm to (133.0, 89.7)
- moved C13 4.69 mm to (152.9, 89.0)
- moved C12 2.49 mm to (145.2, 89.0)
- moved C8 0.71 mm to (135.4, 84.3)
- moved C9 0.70 mm to (133.5, 84.3)
- moved RST2 0.47 mm to (70.4, 84.8)
- moved C22 0.42 mm to (79.6, 77.6), turned to 180 degrees
- moved BUT2 0.42 mm to (70.4, 91.6)
- moved C21 0.37 mm to (79.7, 75.8), turned to 0 degrees
- renumbered C8 to C10, C9 to C11, C10 to C12, C11 to C13, C12 to C14, C13 to C15, C18 to C16, C16 to C17, C17 to C18, C22 to C20, C19 to C21, C14 to C3, C15 to C4, C6 to C8, C7 to C9, D8 to D10, D9 to D11, D10 to D12, D11 to D13, D12 to D14, D2 to D4, D3 to D5, D4 to D6, D5 to D7, D6 to D8, D7 to D9, R10 to R11, R9 to R12, R15 to R13, R13 to R14, R14 to R15, R5 to R2, R3 to R4, R4 to R5, R11 to R7, R7 to R9, U4 to U3, U3 to U4
Connections:
- J2 pad 1: +24V -> Net-(J2-Pin_1)
Routing:
- net +3.3V: track 81.2 -> 39.0 mm
- net GND: track 16.4 -> 4.87 mm, vias 80 -> 81
- net Net-(D2-A): track 0.00 -> 3.98 mm
- net /TOP/MCU&LEDS/LED_SPI_MOSI: track 12.8 -> 15.7 mm
- net Net-(J2-Pin_1): track 0.00 -> 2.87 mm
- net Net-(Q2-D): track 0.00 -> 2.26 mm
- net /TOP/MCU&LEDS/LED_SPI_CLK: track 13.0 -> 11.6 mm
- net +5V: track 43.1 -> 42.4 mm
- net /TOP/MCU&LEDS/GPIO11\FSPID(SPI3_MOSI): track 25.4 -> 26.1 mm
- net Net-(BUT2-~-Pad1): track 6.11 -> 6.75 mm

Commit message: PCB redesign
Parts:
- added C5: 4.7uF/50V/X7R/1210, Capacitor_SMD:C_1210_3225Metric, B.Cu at (150.1, 76.3)
- added C6: 4.7uF/50V/X7R/1210, Capacitor_SMD:C_1210_3225Metric, B.Cu at (153.4, 76.3)
- C20: renamed from C19; footprint Capacitor_Tantalum_SMD:CP_EIA-2012-12_Kemet-R_HandSolder -> Capacitor_SMD:C_0603_1608Metric
- C22: footprint Capacitor_Tantalum_SMD:CP_EIA-2012-12_Kemet-R_HandSolder -> Capacitor_SMD:C_0603_1608Metric
- C7: renamed from C6; value 4.7uF/50V -> 100uF/50V; footprint Capacitor_SMD:CP_Elec_4x5.7 -> Capacitor_SMD:CP_Elec_8x10.5
- C8: renamed from C7; value 4.7uF/50V -> 4.7uF/50V/X7R/1210; footprint Capacitor_SMD:CP_Elec_4x5.7 -> Capacitor_SMD:C_1210_3225Metric
- L2: value 4.7uH -> 4.7uH/MWSA1003S
- moved C9 8.98 mm to (139.7, 76.4), turned to -90 degrees
- moved R8 4.23 mm to (137.3, 76.2), turned to -90 degrees
- moved C8 3.58 mm to (142.2, 76.4)
- moved R6 3.40 mm to (152.7, 83.3), turned to 180 degrees
- moved D2 2.91 mm to (149.7, 81.1)
- moved Q2 2.84 mm to (152.8, 80.7)
- moved D3 2.66 mm to (146.1, 77.0)
- moved C14 2.06 mm to (155.0, 89.2)
- moved F2 1.98 mm to (156.4, 80.6), turned to -90 degrees
- moved C13 1.91 mm to (147.1, 89.2)
- moved C12 1.45 mm to (133.3, 89.7)
- moved C11 1.41 mm to (131.6, 89.7)
- moved C10 0.30 mm to (133.2, 84.3)
- moved C23 0.13 mm to (79.6, 75.8)
- renumbered C9 to C10, C10 to C11, C11 to C12, C12 to C13, C13 to C14, C14 to C15, C15 to C16, C16 to C17, C17 to C18, C18 to C19, C20 to C21, C21 to C23, C8 to C9
Connections:
- net /TOP/MCU&LEDS/GPIO0\BUT1 renamed /TOP/MCU&LEDS/GPIO0_BUT1
- net /TOP/MCU&LEDS/GPIO11\FSPID(SPI3_MOSI) renamed /TOP/MCU&LEDS/GPIO11_FSPID_SPI3_MOSI
- net /TOP/MCU&LEDS/GPIO12\FSPICLK(SPI3_CLK) renamed /TOP/MCU&LEDS/GPIO12_FSPICLK_SPI3_CLK
- net /TOP/MCU&LEDS/GPIO19\USB_D- renamed /TOP/MCU&LEDS/GPIO19_USB_DM
- net /TOP/MCU&LEDS/GPIO20\USB_D+ renamed /TOP/MCU&LEDS/GPIO20_USB_DP
- net /TOP/MCU&LEDS/GPIO5\PWR_SENS renamed /TOP/MCU&LEDS/GPIO5_PWR_SENS
Routing:
- net GND: track 4.87 -> 2.28 mm, vias 81 -> 80
- net Net-(Q2-D): track 2.26 -> 3.19 mm

Commit message: PCB redesign
Parts:
- added C24: 100nF/50V/0603, Capacitor_SMD:C_0603_1608Metric, F.Cu at (95.0, 105.6)
- added R16: 10k/R0603, Resistor_SMD:R_0603_1608Metric_Pad0.98x0.95mm_HandSolder, F.Cu at (87.2, 102.4)

Commit message: PCB redesign
Parts:
- renumbered R16 to R13, R13 to R14, R14 to R15, R15 to R16
